File: Sinister/Sinister.kicad_pcb (KiCad board)
At the start: 2 copper layers, 426 parts, among them J1 TYPE-C-31-M12_13, J2 Conn_ARM_JTAG_SWD_10, Q1 AO3401A, Q2 DTC123JKAT146, Q3 DTC123JKAT146, Q4 AO3401A, SW1 MINUS, SW10 4, SW11 5, SW12 6, SW13 7, SW14 8, SW15 9, SW16 0, SW17 MINUS, SW18 PLUS, SW19 BKSP, SW2 FSLASH, SW20 NUM 7, SW21 NUM 8, SW22 NUM 9, SW23 END, SW24 TAB, SW25 Q, SW26 W, SW27 E, SW28 R, SW29 T, SW3 ASTERISK, SW30 Y, SW31 U, SW32 I, SW33 O, SW34 P, SW35 LBRKT, SW36 RBRKT, SW37 BSLASH, SW38 NUM PLUS, SW39 NUM4, SW4 NUM LOCK, SW40 NUM5, SW41 NUM 6, SW42 DEL, SW43 CAPSLOCK, SW44 A, SW45 S, SW46 D, SW47 F, SW48 G, SW49 H, SW5 HOME, SW50 J, SW51 K, SW52 L, SW53 COLON, SW54 QUOTE, SW55 ENTER, SW56 NUM 1, SW57 NUM 2, SW58 NUM 3, SW59 UP, SW6 ESC, SW60 LSHIFT, SW61 Z, SW62 X, SW63 C, SW64 V, SW65 B, SW66 N, SW67 M, SW68 COMMA, SW69 PERIOD, SW7 1, SW70 FSLASH, SW71 RSHIFT, SW72 NUM ENTER, SW73 NUM PERIOD, SW74 NUM 0, SW75 LEFT, SW76 DOWN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

Commit message: pushed for Gondo Help
Trying to length match USBC data lines
Parts:
- SW80: footprint acheron_MX:MX625 -> acheron_MX:MX625R
- U3: footprint Package_SON:USON-10_2.5x1.0mm_P0.5mm -> acheron_Components:USON-10_2.5x1.0mm_P0.5mm
- moved D103 219.7 mm to (215.4, 100.0)
- moved U3 198.2 mm to (269.1, 26.3)
- moved J1 193.3 mm to (269.1, 24.1), turned to 0 degrees
- moved D95 193.3 mm to (507.1, 42.9), turned to 180 degrees
- moved D97 179.7 mm to (507.1, 100.0)
- moved D89 174.9 mm to (215.4, 42.9), turned to 180 degrees
- moved D93 144.5 mm to (409.8, 42.9), turned to 180 degrees
- moved D88 130.0 mm to (205.0, 72.6), turned to -90 degrees
- moved D91 129.2 mm to (312.6, 42.9), turned to 180 degrees
- moved D102 127.3 mm to (266.5, 100.0)
- moved U1 125.6 mm to (273.4, 78.0), turned to 135 degrees
- moved D96 124.4 mm to (517.4, 72.6), turned to 90 degrees
- moved D92 119.1 mm to (361.2, 42.9), turned to 180 degrees
- moved D90 116.3 mm to (264.0, 42.9), turned to 180 degrees
- moved D94 112.4 mm to (458.4, 42.9), turned to 180 degrees
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Connections:
- U3 pad 1: D+ -> D-
- U3 pad 10: D+ -> D-
- U3 pad 2: D- -> D+
- U3 pad 9: D- -> D+
Routing:
- net D-: track 0.00 -> 59.1 mm, vias 0 -> 3
- net D+: track 0.00 -> 58.6 mm, vias 0 -> 3
- net (no net): track 0.00 -> 2.70 mm
Other:
- board outline added: 386.8 x 104.7 mm

Commit message: Began placing and routing power and RGB components.
Placed and routed: RGB caps and resistors, MCU caps, VBUS components.
Parts:
- R65, R66: footprint Resistor_SMD:R_0402_1005Metric -> acheron_Components:R_SMD_1206
- SW60: moved to F.Cu
- moved C16 239.3 mm to (224.3, 40.2), turned to 90 degrees
- moved C15 208.9 mm to (204.5, 64.1), turned to 0 degrees
- moved R65 201.5 mm to (264.1, 26.6), turned to 90 degrees
- moved R97 194.8 mm to (221.9, 39.8)
- moved R96 193.2 mm to (204.9, 66.5), turned to 180 degrees
- moved F1 189.3 mm to (265.5, 34.8)
- moved C13 188.6 mm to (261.9, 26.1)
- moved R24 187.8 mm to (266.8, 26.3)
- moved D87 187.4 mm to (268.9, 35.3), turned to 90 degrees
- moved C14 187.3 mm to (277.2, 25.0), turned to 0 degrees
- moved R98 173.7 mm to (281.6, 39.8)
- moved C17 169.8 mm to (284.0, 40.3), turned to 90 degrees
- moved R100 156.6 mm to (366.1, 39.8)
- moved R66 156.1 mm to (274.0, 26.4), turned to 90 degrees
- moved C1 149.9 mm to (280.2, 77.7), turned to 45 degrees
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Routing:
- net Net-(D90-Pad2): track 0.00 -> 45.7 mm
- net Net-(D92-Pad2): track 0.00 -> 45.6 mm
- net Net-(D91-Pad2): track 0.00 -> 45.6 mm
- net Net-(D89-Pad2): track 0.00 -> 45.6 mm
- net Net-(D88-Pad2): track 0.00 -> 35.2 mm, vias 0 -> 2
- net Net-(C13-Pad1): track 0.00 -> 28.4 mm
- net 3V3: track 0.00 -> 22.0 mm, vias 0 -> 1
- net Net-(Q1-Pad3): track 1793.1 -> 1811.4 mm, vias 0 -> 4
- net Net-(C17-Pad1): track 0.00 -> 17.6 mm
- net Row0: track 387.3 -> 404.6 mm, vias 0 -> 4
- net VBUS: track 0.00 -> 16.9 mm, vias 0 -> 2
- net 5V: track 0.00 -> 8.23 mm
- net Net-(C18-Pad1): track 0.00 -> 6.99 mm
- net Net-(C16-Pad1): track 0.00 -> 6.50 mm
- net Net-(C15-Pad1): track 0.00 -> 6.05 mm, vias 0 -> 2
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
Commit message: Placed and routed reaminder of RGB components.
Repositioned RGB components, rereouted RGB connections. Rerouted Columns.
Parts:
- SW60: moved to B.Cu
- moved R103 280.1 mm to (511.9, 42.8), turned to 90 degrees
- moved R107 254.2 mm to (521.6, 73.6)
- moved C22 236.1 mm to (515.2, 41.3), turned to 0 degrees
- moved C24 215.3 mm to (508.6, 105.1), turned to 0 degrees
- moved C20 210.3 mm to (418.0, 41.3), turned to 0 degrees
- moved R104 210.0 mm to (204.9, 77.9), turned to 180 degrees
- moved R108 206.6 mm to (505.4, 106.6), turned to 90 degrees
- moved C25 190.0 mm to (459.3, 105.1), turned to 0 degrees
- moved R114 188.6 mm to (206.5, 106.6), turned to 90 degrees
- moved R101 177.1 mm to (414.7, 42.8), turned to 90 degrees
- moved C26 158.2 mm to (413.3, 105.1), turned to 0 degrees
- moved R106 150.1 mm to (203.7, 81.7), turned to 90 degrees
- moved C23 141.3 mm to (523.8, 74.1), turned to 90 degrees
- moved C21 138.5 mm to (466.6, 41.3), turned to 0 degrees
- moved R102 137.8 mm to (463.3, 42.8), turned to 90 degrees
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Connections:
- R110 pad 1: 5V -> Net-(C26-Pad1)
- R110 pad 2: Net-(C26-Pad1) -> 5V
- SW80 pad 1: COL9 -> COL10
- U1 pad 28: Net-(U1-Pad28) -> RGB_3V3
Routing:
- net 5V: track 8.23 -> 160.5 mm, vias 0 -> 3
- net RGB_3V3: track 0.00 -> 72.7 mm
- net Net-(D102-Pad2): track 0.00 -> 49.3 mm
- net Net-(D98-Pad2): track 0.00 -> 45.6 mm
- net Net-(D93-Pad2): track 0.00 -> 45.6 mm
- net Net-(D100-Pad2): track 0.00 -> 45.6 mm
- net Net-(D97-Pad2): track 0.00 -> 45.6 mm
- net Net-(D100-Pad4): track 0.00 -> 45.6 mm
- net Net-(D94-Pad2): track 0.00 -> 45.6 mm
- net Net-(D101-Pad2): track 0.00 -> 45.2 mm
- net COL9: track 121.5 -> 80.9 mm
- net RGB8-RGB9: track 0.00 -> 35.2 mm, vias 0 -> 2
- net Net-(D96-Pad2): track 0.00 -> 32.6 mm, vias 0 -> 2
- net COL10: track 81.0 -> 102.3 mm
- net Net-(C17-Pad1): track 17.6 -> 4.70 mm
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
Commit message: Rereouted diodes. Placed LED components.
Replaced diodes tracks. Placed and routed LED power components. Routed 5V RGB tracks.
Parts:
- moved Q1 130.9 mm to (210.5, 81.5), turned to 180 degrees
- moved R2 130.1 mm to (213.6, 81.0), turned to 90 degrees
- moved R3 130.0 mm to (216.2, 81.0), turned to 90 degrees
- moved Q2 113.7 mm to (219.3, 81.5), turned to 180 degrees
- moved J2 87.3 mm to (278.7, 92.1), turned to -90 degrees
- moved R99 2.19 mm to (317.5, 42.8)
- moved C18 2.19 mm to (320.8, 41.3)
- turned R110 to -90 degrees
Connections:
- net Row0 renamed ROW0
- SW82 pad 1: COL14 -> COL15
- SW83 pad 1: COL15 -> COL16
- SW84 pad 1: COL16 -> COL17
- U1 pad 16: Net-(U1-Pad16) -> LED_PWM
Routing:
- net 5V: track 160.5 -> 864.3 mm, vias 3 -> 8
- net Net-(Q1-Pad3): track 1811.4 -> 1929.2 mm
- net COL17: track 64.3 -> 111.9 mm
- net COL14: track 121.4 -> 80.9 mm
- net COL15: track 126.2 -> 102.3 mm
- net ROW0: track 404.6 -> 397.3 mm
- net ROW1: track 371.5 -> 364.3 mm
- net ROW2: track 378.0 -> 370.9 mm
- net Net-(C18-Pad1): track 6.88 -> 0.00 mm
- net ROW3: track 356.7 -> 350.3 mm
- net Net-(Q1-Pad1): track 0.00 -> 6.35 mm
- net Net-(Q2-Pad3): track 0.00 -> 6.06 mm
- net ROW4: track 380.5 -> 375.6 mm
- net COL16: track 131.0 -> 126.2 mm
- net Net-(D5-Pad2): track 0.00 -> 3.08 mm
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