File: Sinister/sinister.kicad_sch (KiCad schematic)
At the start: 177 parts, among them SW1 MINUS, SW10 4, SW11 5, SW12 6, SW13 7, SW14 8, SW15 9, SW16 0, SW17 MINUS, SW18 PLUS, SW19 BKSP, SW2 FSLASH, SW21 NUM 7, SW22 NUM 8, SW23 NUM 9, SW24 END, SW25 TAB, SW26 Q, SW27 W, SW28 E, SW29 R, SW3 ASTERISK, SW30 T, SW31 Y, SW32 U, SW33 I, SW34 O, SW35 P, SW36 LBRKT, SW37 RBRKT, SW38 BSLASH, SW39 NUM PLUS, SW4 NUM LOCK, SW40 NUM4, SW41 NUM5, SW42 NUM 6, SW43 DEL, SW44 CAPSLOCK, SW45 A, SW46 S, SW47 D, SW48 F, SW49 G, SW5 HOME, SW50 H, SW51 J, SW52 K, SW53 L, SW54 COLON, SW55 QUOTE, SW56 ENTER, SW58 NUM 1, SW59 NUM 2, SW6 ESC, SW60 NUM 3, SW61 UP, SW62 LSHIFT, SW63 Z, SW64 X, SW65 C, SW66 V, SW67 B, SW68 N, SW69 M, SW7 1, SW70 COMMA, SW71 PERIOD, SW72 FSLASH, SW73 RSHIFT, SW77 NUM ENTER, SW78 NUM PERIOD, SW79 NUM 0, SW8 2, SW80 LEFT, SW81 DOWN, SW82 RIGHT, SW83 LCTRL, SW84 LALT, SW87 SPACE, SW9 3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

Commit message: Added ancilliary components to schematic.
Added the LED array, USB connector, ESD protection, MCU reset circuit, LDO, and JTAG SWD. Added and connected necessary components for the MCU.
Parts:
- added C? (x2): 4.7u, Capacitor_SMD:C_0402_1005Metric, symbol Device:C_Small
- added C? (x2): 1u, Capacitor_SMD:C_0805_2012Metric_Pad1.15x1.40mm_HandSolder, symbol Device:C_Small
- added C? (x4): 100n, Capacitor_SMD:C_0402_1005Metric, symbol Device:C_Small
- added C?: 100u, Capacitor_SMD:C_0805_2012Metric_Pad1.15x1.40mm_HandSolder, symbol Device:C_Small
- added C?: 1u, Capacitor_SMD:C_0402_1005Metric, symbol Device:C_Small
- added C?: 10n, Capacitor_SMD:C_0402_1005Metric, symbol Device:C_Small
- added C?: 10u, Capacitor_SMD:C_0805_2012Metric_Pad1.15x1.40mm_HandSolder, symbol Device:C_Small
- added D?: RB060M-60TR, acheron_Components:D_SOD-123, symbol Device:D_Schottky_Small
- added D?: SMF9.0CA, acheron_Components:D_SOD-123_Bidirectional, symbol Device:D_TVS
- added D?: 1N4148W, acheron_Components:D_SOD-123, symbol Device:D_Small
- added F?: RF1338-000, Fuse:Fuse_1812_4532Metric_Pad1.30x3.40mm_HandSolder, symbol Device:Polyfuse_Small
- added J?: Conn_ARM_JTAG_SWD_10, acheron_Connectors:Conn_ARM_JTAG_SWD_10, symbol acheronSymbols:Conn_ARM_JTAG_SWD_10
- added LED? (x84): LED, acheron_Components:LED_THT_2.54mm, symbol acheronSymbols:LED
- added Q? (x2): DTC123JKAT146, Package_TO_SOT_SMD:SOT-23, symbol Transistor_BJT:DTC123J
- added Q?: AO3401A, Package_TO_SOT_SMD:SOT-23, symbol Transistor_FET:AO3401A
- added R? (x2): 100R, acheron_Components:R_SMD_1206, symbol Device:R_Small
- added R? (x84): 390R, acheron_Components:R_SMD_1206, symbol Device:R_Small
- added R?: 33k, acheron_Components:R_SMD_1206, symbol Device:R_Small
- added R?: 10k, acheron_Components:R_SMD_1206, symbol Device:R_Small
- added R? (x3): 100k, acheron_Components:R_SMD_1206, symbol Device:R_Small
- added SW?: K2-1187SQ-A4SW-06, acheron_Hardware:K2-1187SQ-A4SW-06, symbol Switch:SW_Push
- added U?: MCP1700-3302E_SOT23, Package_TO_SOT_SMD:SOT-23, symbol Regulator_Linear:MCP1700-3302E_SOT23
- C? (x2): value 100nF -> 100n; footprint (none) -> Capacitor_SMD:C_0805_2012Metric_Pad1.15x1.40mm_HandSolder; PACKAGE (none) -> C0805
- SW25, SW83: footprint acheron_MX:MX100 -> acheron_MX:MX150
- SW38: footprint acheron_MX:MX200 -> acheron_MX:MX150
- SW39, SW77: footprint acheron_MX:MX100 -> acheron_MX:MX200V
- SW44: footprint acheron_MX:MX100 -> acheron_MX:MX175
- SW56: footprint acheron_MX:MX100 -> acheron_MX:MX225
- SW62: footprint acheron_MX:MX100 -> acheron_MX:MX225R
- SW73: footprint acheron_MX:MX100 -> acheron_MX:MX275R
- SW84, SW90, SW91, SW92, SW93: footprint acheron_MX:MX100 -> acheron_MX:MX125
- SW87: footprint acheron_MX:MX100 -> acheron_MX:MX625
Connections:
- net D+: now also U?.33 (USB_DP/PA12)
- net D-: now also U?.32 (USB_DM/TIM1_CH4/PA11)
- net GND: now also U?.23 (VSS), U?.35 (VSS), U?.47 (VSS), U?.8 (VSSA), C?.1, C?.1, C?.1, C?.1, C?.1, C?.1, C?.1, C?.2, C?.2, C?.2, C?.2, C?.2, D?.2 (A2), J?.3 (GND), J?.5 (GND), J?.9 (GNDDetect), LED?.K, LED?.K, LED?.K, LED?.K, LED?.K, LED?.K, LED?.K, LED?.K, LED?.K, LED?.K, LED?.K, LED?.K, LED?.K, LED?.K, LED?.K, LED?.K, LED?.K, LED?.K, LED?.K, LED?.K, LED?.K, LED?.K, LED?.K, LED?.K, LED?.K, LED?.K, LED?.K, LED?.K, LED?.K, LED?.K, LED?.K, LED?.K, LED?.K, LED?.K, LED?.K, LED?.K, LED?.K, LED?.K, LED?.K, LED?.K, LED?.K, LED?.K, LED?.K, LED?.K, LED?.K, LED?.K, LED?.K, LED?.K, LED?.K, LED?.K, LED?.K, LED?.K, LED?.K, LED?.K, LED?.K, LED?.K, LED?.K, LED?.K, LED?.K, LED?.K, LED?.K, LED?.K, LED?.K, LED?.K, LED?.K, LED?.K, LED?.K, LED?.K, LED?.K, LED?.K, LED?.K, LED?.K, LED?.K, LED?.K, LED?.K, LED?.K, LED?.K, LED?.K, LED?.K, LED?.K, LED?.K, LED?.K, LED?.K, LED?.K, Q?.2 (E), Q?.2 (E), R?.2, R?.2, R?.2, U?.1 (GND)
- net VBUS: now also F?.1
- net 3V3: now reaches U?.1 (VBAT)
- net 3V3: now also U?.24 (VDD), U?.36 (VDDIO2), U?.48 (VDD), U?.9 (VDDA), C?.1, C?.1, C?.2, C?.2, C?.2, C?.2, C?.2, C?.2, C?.2, D?.2 (A), J?.1 (VCC), R?.1, SW?.1, U?.2 (VO)
- net SWDIO: now reaches U?.34 (SWDIO/PA13)
- net SWDIO: now also J?.2 (SWDIO/TMS)
- net SWCLK: now reaches U?.37 (SWCLK/PA14)
- net SWCLK: now also J?.4 (SWDCLK/TCK)
- net BOOT0: now reaches U?.44 (BOOT0)
- net BOOT0: now also C?.1, R?.1, R?.1
- net nRST: now reaches U?.7 (NRST)
- net nRST: now also C?.1, J?.10 (~RESET~), R?.2
- new net: Q?.1 (G), R?.1
- new net: Q?.3 (C), R?.2, R?.2
- new net: LED?.A, R?.1 (x84)
- new net: Q?.3 (D), R?.2, R?.2, R?.2, R?.2, R?.2, R?.2, R?.2, R?.2, R?.2, R?.2, R?.2, R?.2, R?.2, R?.2, R?.2, R?.2, R?.2, R?.2, R?.2, R?.2, R?.2, R?.2, R?.2, R?.2, R?.2, R?.2, R?.2, R?.2, R?.2, R?.2, R?.2, R?.2, R?.2, R?.2, R?.2, R?.2, R?.2, R?.2, R?.2, R?.2, R?.2, R?.2, R?.2, R?.2, R?.2, R?.2, R?.2, R?.2, R?.2, R?.2, R?.2, R?.2, R?.2, R?.2, R?.2, R?.2, R?.2, R?.2, R?.2, R?.2, R?.2, R?.2, R?.2, R?.2, R?.2, R?.2, R?.2, R?.2, R?.2, R?.2, R?.2, R?.2, R?.2, R?.2, R?.2, R?.2, R?.2, R?.2, R?.2, R?.2, R?.2, R?.2, R?.2, R?.2
- new net: D?.1 (K), R?.2
- new net: D?.2 (A), Q?.1 (B), SW?.2
- new net: Q?.3 (C), R?.1
- new net 5V: C?.1, D?.1 (A1), D?.1 (K), F?.2, Q?.2 (S), R?.1, R?.1, U?.3 (VI)
- new net LED_PWM: Q?.1 (B)
- no-connect marks 2 -> 4
Other:
- note added: "ESD Protection"
- note added: "JTAG SWD"
- note added: "LDO"
- note added: "LEDs"
- note added: "MCU Reset"
- note added: "SWITCH MATRIX"
- note added: "USB Connector"
- moved on the sheet: C?, D1, D10, D11, D12, D13, D14, D15, D16, D17, D18, D19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

Commit message: Placed components and routed matrixes.
Placed LED resistors and keyswitch diodes. Routed LED and keyswitch matrixes. Repositioned labels for clarity and organization.
Parts:
- added C15, C16, C17, C18, C19, C20, C21, C22, C23, C24, C25, C26, C27, C28, C29, C30: 1u, Capacitor_SMD:C_0805_2012Metric_Pad1.15x1.40mm_HandSolder, symbol Device:C_Small
- added D100, D101, D102, D103, D88, D89, D90, D91, D92, D93, D94, D95, D96, D97, D98, D99: WS2812C, acheron_Components:LED_WS2812B_5.0x5.0mm_P3.2mm, symbol LED:WS2812B
- added Q4: AO3401A, Package_TO_SOT_SMD:SOT-23, symbol Transistor_FET:AO3401A
- added R100, R101, R102, R103, R107, R108, R109, R110, R111, R112, R113, R114, R96, R97, R98, R99: 3R, acheron_Components:R_SMD_1206, symbol Device:R_Small
- added R104, R106: 10k, acheron_Components:R_SMD_1206, symbol Device:R_Small
- added R105: 5.1k, acheron_Components:R_SMD_1206, symbol Device:R_Small
- J1: renamed from J?; footprint acheronConnectors:TYPE-C-31-M-12 -> acheron_Connectors:TYPE-C-31-M-12
- SW19: footprint acheron_MX:MX200 -> acheron_MX:MX200R
- SW38: renamed from SW39; footprint acheron_MX:MX200V -> acheron_MX:MX200VR
- SW72: renamed from SW77; footprint acheron_MX:MX200V -> acheron_MX:MX200VR
- gave numbers to parts that had none: 205
- renumbered D21 to D20, D22 to D21, D23 to D22, D24 to D23, D25 to D24, D26 to D25, D27 to D26, D28 to D27, D29 to D28, D30 to D29, D31 to D30, D32 to D31, D33 to D32, D34 to D33, D35 to D34, D36 to D35, D37 to D36, D38 to D37, D39 to D38, D40 to D39, D41 to D40, D42 to D41, D43 to D42, D44 to D43, D45 to D44, D46 to D45, D47 to D46, D48 to D47, D49 to D48, D50 to D49, D51 to D50, D52 to D51, D53 to D52, D54 to D53, D55 to D54, D56 to D55, D58 to D56, D59 to D57, D60 to D58, D61 to D59, D62 to D60, D63 to D61, D64 to D62, D65 to D63, D66 to D64, D67 to D65, D68 to D66, D69 to D67, D70 to D68, D71 to D69, D72 to D70, D73 to D71, D77 to D72, D78 to D73, D79 to D74, D80 to D75, D81 to D76, D82 to D77, D83 to D78, D84 to D79, D87 to D80, D90 to D81, D91 to D82, D92 to D83, D93 to D84, SW21 to SW20, SW22 to SW21, SW23 to SW22, SW24 to SW23, SW25 to SW24, SW26 to SW25, SW27 to SW26, SW28 to SW27, SW29 to SW28, SW30 to SW29, SW31 to SW30, SW32 to SW31, SW33 to SW32, SW34 to SW33, SW35 to SW34, SW36 to SW35, SW37 to SW36, SW38 to SW37, SW40 to SW39, SW41 to SW40, SW42 to SW41, SW43 to SW42, SW44 to SW43, SW45 to SW44, SW46 to SW45, SW47 to SW46, SW48 to SW47, SW49 to SW48, SW50 to SW49, SW51 to SW50, SW52 to SW51, SW53 to SW52, SW54 to SW53, SW55 to SW54, SW56 to SW55, SW58 to SW56, SW59 to SW57, SW60 to SW58, SW61 to SW59, SW62 to SW60, SW63 to SW61, SW64 to SW62, SW65 to SW63, SW66 to SW64, SW67 to SW65, SW68 to SW66, SW69 to SW67, SW70 to SW68, SW71 to SW69, SW72 to SW70, SW73 to SW71, SW78 to SW73, SW79 to SW74, SW80 to SW75, SW81 to SW76, SW82 to SW77, SW83 to SW78, SW84 to SW79, SW87 to SW80, SW90 to SW81, SW91 to SW82, SW92 to SW83, SW93 to SW84
Connections:
- net 5V: now also R100.1, R101.1, R102.1, R103.1, R104.1, R105.1, R107.1, R108.1, R109.1, R110.1, R111.1, R112.1, R113.1, R114.1, R96.1, R97.1, R98.1, R99.1
- net COL10: no longer SW80.1 (Col)
- net COL9: now also SW80.1 (Col)
- net GND: now also C15.2, C16.2, C17.2, C18.2, C19.2, C20.2, C21.2, C22.2, C23.2, C24.2, C25.2, C26.2, C27.2, C28.2, C29.2, C30.2, D100.3 (VSS), D101.3 (VSS), D102.3 (VSS), D103.3 (VSS), D88.3 (VSS), D89.3 (VSS), D90.3 (VSS), D91.3 (VSS), D92.3 (VSS), D93.3 (VSS), D94.3 (VSS), D95.3 (VSS), D96.3 (VSS), D97.3 (VSS), D98.3 (VSS), D99.3 (VSS), R106.2
- new net: Q4.1 (G), R105.2, R106.1
- new net: C21.1, D94.1 (VDD), R102.2
- new net: C24.1, D97.1 (VDD), R108.2
- new net: D97.2 (DOUT), D98.4 (DIN)
- new net: D96.2 (DOUT), D97.4 (DIN)
- new net: C16.1, D89.1 (VDD), R97.2
- new net: D89.2 (DOUT), D90.4 (DIN)
- new net: D88.2 (DOUT), D89.4 (DIN)
- new net: C29.1, D102.1 (VDD), R113.2
- new net: D102.2 (DOUT), D103.4 (DIN)
- new net: D101.2 (DOUT), D102.4 (DIN)
- new net: C19.1, D92.1 (VDD), R100.2
- new net: D92.2 (DOUT), D93.4 (DIN)
- new net: D91.2 (DOUT), D92.4 (DIN)
- new net: C28.1, D101.1 (VDD), R112.2
- new net: C18.1, D91.1 (VDD), R99.2
- new net: C26.1, D99.1 (VDD), R110.2
- new net: D100.4 (DIN), D99.2 (DOUT)
- new net: D98.2 (DOUT), D99.4 (DIN)
- new net: C23.1, D96.1 (VDD), R107.2
- new net: C25.1, D98.1 (VDD), R109.2
- new net: D94.2 (DOUT), D95.4 (DIN)
- new net: D93.2 (DOUT), D94.4 (DIN)
- new net: C27.1, D100.1 (VDD), R111.2
- new net: D100.2 (DOUT), D101.4 (DIN)
- new net: C15.1, D88.1 (VDD), R96.2
- new net: C20.1, D93.1 (VDD), R101.2
- new net: C17.1, D90.1 (VDD), R98.2
- new net: C30.1, D103.1 (VDD), R114.2
- new net: C22.1, D95.1 (VDD), R103.2
- new net: D90.2 (DOUT), D91.4 (DIN)
- new net RGB8-RGB9: D95.2 (DOUT), D96.4 (DIN)
- new net RGB_3V3: Q4.3 (D)
- new net RGB_5V: D88.4 (DIN), Q4.2 (S), R104.2
- no-connect marks 4 -> 5
Other:
- note added: "MCU"
- note added: "RBG"
- moved on the sheet: C1, C10, C11, C12, C2, C3, C4, C5, C6, C7, C8, C9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

Commit message: pushed for Gondo Help
Trying to length match USBC data lines
Parts:
- SW80: footprint acheron_MX:MX625 -> acheron_MX:MX625R
- U3: footprint Package_SON:USON-10_2.5x1.0mm_P0.5mm -> acheron_Components:USON-10_2.5x1.0mm_P0.5mm
Connections:
- net D+: now also U3.2 (IO2), U3.9 (NC); no longer U3.1 (IO1), U3.10 (NC)
- net D-: now also U3.1 (IO1), U3.10 (NC); no longer U3.2 (IO2), U3.9 (NC)
Changed lines of the file:
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@@
   (junction (at 528.574 36.576) (diameter 0) (color 0 0 0 0))
   (junction (at 528.574 42.926) (diameter 0) (color 0 0 0 0))
+  (no_connect (at 227.076 368.046))
   (no_connect (at 279.4 231.14))
-  (no_connect (at 279.4 233.68))
-  (no_connect (at 320.04 278.638))
   (no_connect (at 320.04 281.178))
-  (no_connect (at 227.076 368.046))
+  (no_connect (at 320.04 278.638))
+  (no_connect (at 279.4 233.68))
   (wire (pts (xy 20.32 334.264) (xy 29.21 334.264))
     (stroke (width 0) (type solid) (color 0 0 0 0))
@@
     (effects (font (size 0.75 0.75)) (justify left))
   )
-  (global_label "D+" (shape bidirectional) (at 256.286 279.4 180)
+  (global_label "D-" (shape bidirectional) (at 256.286 279.4 180)
     (effects (font (size 0.75 0.75)) (justify right))
   )
-  (global_label "D+" (shape bidirectional) (at 256.286 281.94 180)
+  (global_label "D-" (shape bidirectional) (at 256.286 281.94 180)
     (effects (font (size 0.75 0.75)) (justify right))
   )
-  (global_label "D-" (shape bidirectional) (at 256.286 287.02 180)
+  (global_label "D+" (shape bidirectional) (at 256.286 287.02 180)
     (effects (font (size 0.75 0.75)) (justify right))
   )
-  (global_label "D-" (shape bidirectional) (at 256.286 289.56 180)
+  (global_label "D+" (shape bidirectional) (at 256.286 289.56 180)
     (effects (font (size 0.75 0.75)) (justify right))
   )
@@
       (effects (font (size 0.991 0.991)))
     )
-    (property "Footprint" "acheron_MX:MX625" (id 2) (at 214.376 151.892 0)
+    (property "Footprint" "acheron_MX:MX625R" (id 2) (at 214.376 151.892 0)
       (effects (font (size 1.27 1.27)) hide)
     )
@@
     (property "Reference" "U3" (id 0) (at 268.986 272.6498 0))
     (property "Value" "TPD4E05U06DQAR" (id 1) (at 268.986 274.9485 0))
-    (property "Footprint" "Package_SON:USON-10_2.5x1.0mm_P0.5mm" (id 2) (at 268.986 257.81 0)
+    (property "Footprint" "acheron_Components:USON-10_2.5x1.0mm_P0.5mm" (id 2) (at 268.986 257.81 0)
       (effects (font (size 1.27 1.27)) hide)
     )

Commit message: Began placing and routing power and RGB components.
Placed and routed: RGB caps and resistors, MCU caps, VBUS components.
Parts:
- R65, R66: footprint Resistor_SMD:R_0402_1005Metric -> acheron_Components:R_SMD_1206
Changed lines of the file:
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@@
   (junction (at 528.574 36.576) (diameter 0) (color 0 0 0 0))
   (junction (at 528.574 42.926) (diameter 0) (color 0 0 0 0))
+  (no_connect (at 279.4 233.68))
   (no_connect (at 227.076 368.046))
-  (no_connect (at 279.4 231.14))
   (no_connect (at 320.04 281.178))
   (no_connect (at 320.04 278.638))
-  (no_connect (at 279.4 233.68))
+  (no_connect (at 279.4 231.14))
   (wire (pts (xy 20.32 334.264) (xy 29.21 334.264))
     (stroke (width 0) (type solid) (color 0 0 0 0))
@@
       (effects (font (size 0.75 0.75)))
     )
-    (property "Footprint" "Resistor_SMD:R_0402_1005Metric" (id 2) (at 256.54 254 0)
+    (property "Footprint" "acheron_Components:R_SMD_1206" (id 2) (at 256.54 254 0)
       (effects (font (size 1.27 1.27)) hide)
     )
@@
       (effects (font (size 0.75 0.75)))
     )
-    (property "Footprint" "Resistor_SMD:R_0402_1005Metric" (id 2) (at 272.542 254 0)
+    (property "Footprint" "acheron_Components:R_SMD_1206" (id 2) (at 272.542 254 0)
       (effects (font (size 1.27 1.27)) hide)
     )

Commit message: Placed and routed reaminder of RGB components.
Repositioned RGB components, rereouted RGB connections. Rerouted Columns.
Connections:
- net 5V: now also R110.2; no longer R110.1
- net COL10: now also SW80.1 (Col)
- net COL9: no longer SW80.1 (Col)
- net RGB_3V3: now also U1.28 (SPI2_MOSI/I2S2_SD/PB15)
- net at C26.1, D99.1 (VDD): now also R110.1; no longer R110.2
- no-connect marks 5 -> 6
Other:
- moved on the sheet: D80, R110, SW80
Changed lines of the file:
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@@
   (junction (at 205.486 68.072) (diameter 0) (color 0 0 0 0))
   (junction (at 205.486 96.012) (diameter 0) (color 0 0 0 0))
-  (junction (at 205.486 123.952) (diameter 0) (color 0 0 0 0))
   (junction (at 211.328 183.388) (diameter 0) (color 0 0 0 0))
   (junction (at 211.328 208.788) (diameter 0) (color 0 0 0 0))
@@
   (junction (at 214.376 81.28) (diameter 0) (color 0 0 0 0))
   (junction (at 214.376 109.22) (diameter 0) (color 0 0 0 0))
-  (junction (at 214.376 137.16) (diameter 0) (color 0 0 0 0))
   (junction (at 219.456 320.802) (diameter 0) (color 0 0 0 0))
   (junction (at 219.456 359.156) (diameter 0) (color 0 0 0 0))
@@
   (junction (at 225.806 68.072) (diameter 0) (color 0 0 0 0))
   (junction (at 225.806 96.012) (diameter 0) (color 0 0 0 0))
+  (junction (at 225.806 123.952) (diameter 0) (color 0 0 0 0))
   (junction (at 231.648 183.388) (diameter 0) (color 0 0 0 0))
   (junction (at 234.696 25.4) (diameter 0) (color 0 0 0 0))
@@
   (junction (at 234.696 81.28) (diameter 0) (color 0 0 0 0))
   (junction (at 234.696 109.22) (diameter 0) (color 0 0 0 0))
+  (junction (at 234.696 137.16) (diameter 0) (color 0 0 0 0))
   (junction (at 246.126 40.132) (diameter 0) (color 0 0 0 0))
   (junction (at 246.126 68.072) (diameter 0) (color 0 0 0 0))
@@
   (junction (at 528.574 42.926) (diameter 0) (color 0 0 0 0))
   (no_connect (at 279.4 233.68))
+  (no_connect (at 517.144 100.076))
   (no_connect (at 227.076 368.046))
-  (no_connect (at 320.04 281.178))
   (no_connect (at 320.04 278.638))
+  (no_connect (at 320.04 281.178))
   (no_connect (at 279.4 231.14))
   (wire (pts (xy 20.32 334.264) (xy 29.21 334.264))
@@
     (stroke (width 0) (type solid) (color 0 0 0 0))
   )
-  (wire (pts (xy 173.736 137.16) (xy 214.376 137.16))
+  (wire (pts (xy 173.736 137.16) (xy 234.696 137.16))
     (stroke (width 0) (type solid) (color 0 0 0 0))
   )
@@
     (stroke (width 0) (type solid) (color 0 0 0 0))
   )
-  (wire (pts (xy 205.486 123.952) (xy 205.486 151.892))
-    (stroke (width 0) (type solid) (color 0 0 0 0))
-  )
   (wire (pts (xy 211.328 183.388) (xy 221.488 183.388))
     (stroke (width 0) (type solid) (color 0 0 0 0))
@@
     (stroke (width 0) (type solid) (color 0 0 0 0))
   )
-  (wire (pts (xy 214.376 137.16) (xy 295.656 137.16))
-    (stroke (width 0) (type solid) (color 0 0 0 0))
-  )
-  (wire (pts (xy 214.376 142.24) (xy 214.376 143.002))
-    (stroke (width 0) (type solid) (color 0 0 0 0))
-  )
   (wire (pts (xy 219.456 313.182) (xy 219.456 314.452))
     (stroke (width 0) (type solid) (color 0 0 0 0))
@@
     (stroke (width 0) (type solid) (color 0 0 0 0))
   )
+  (wire (pts (xy 225.806 123.952) (xy 225.806 151.892))
+    (stroke (width 0) (type solid) (color 0 0 0 0))
+  )
   (wire (pts (xy 225.806 320.802) (xy 227.076 320.802))
     (stroke (width 0) (type solid) (color 0 0 0 0))
@@
     (stroke (width 0) (type solid) (color 0 0 0 0))
   )
+  (wire (pts (xy 234.696 137.16) (xy 295.656 137.16))
+    (stroke (width 0) (type solid) (color 0 0 0 0))
+  )
+  (wire (pts (xy 234.696 142.24) (xy 234.696 143.002))
+    (stroke (width 0) (type solid) (color 0 0 0 0))
+  )
   (wire (pts (xy 241.808 188.468) (xy 241.808 189.738))
     (stroke (width 0) (type solid) (color 0 0 0 0))
@@
     (effects (font (size 1.27 1.27)) (justify left))
   )
+  (global_label "RGB_3V3" (shape output) (at 517.144 87.376 0)
+    (effects (font (size 1.27 1.27)) (justify left))
+  )
   (global_label "3V3" (shape input) (at 531.368 36.576 0)
     (effects (font (size 1.27 1.27)) (justify left))
@@
     )
   )
-  (symbol (lib_id "Device:R_Small") (at 128.016 355.346 0) (unit 1)
+  (symbol (lib_id "Device:R_Small") (at 128.016 355.346 180) (unit 1)
     (in_bom yes) (on_board yes)
-    (property "Reference" "R110" (id 0) (at 125.984 354.584 0)
+    (property "Reference" "R110" (id 0) (at 130.048 356.108 0)
       (effects (font (size 0.75 0.75)))
     )
-    (property "Value" "3R" (id 1) (at 125.984 355.854 0)
+    (property "Value" "3R" (id 1) (at 130.048 354.838 0)
       (effects (font (size 0.75 0.75)))
     )
@@
     )
   )
-  (symbol (lib_id "Device:D_Small") (at 214.376 139.7 270) (unit 1)
-    (in_bom yes) (on_board yes)
-    (property "Reference" "D80" (id 0) (at 216.154 139.7 90)
-      (effects (font (size 0.75 0.75)) (justify left))
-    )
-    (property "Value" "1N4148W" (id 1) (at 216.154 140.849 90)
-      (effects (font (size 0.75 0.75)) (justify left))
-    )
-    (property "Footprint" "acheron_Components:D_SOD-123" (id 2) (at 214.376 139.7 90)
-      (effects (font (size 1.27 1.27)) hide)
-    )
-    (property "Datasheet" "~" (id 3) (at 214.376 139.7 90)
-      (effects (font (size 1.27 1.27)) hide)
-    )
-    (property "MANUFACTURER" "" (id 4) (at 214.376 139.7 90)
-      (effects (font (size 1.27 1.27)) hide)
-    )
-    (property "MANUFACTURER PART NUMBER" "" (id 5) (at 214.376 139.7 90)
-      (effects (font (size 1.27 1.27)) hide)
-    )
-    (property "PACKAGE" "SOD-123" (id 6) (at 214.376 139.7 90)
-      (effects (font (size 1.27 1.27)) hide)
-    )
-    (property "LCSC PART NUMBER" "" (id 7) (at 214.376 139.7 90)
-      (effects (font (size 1.27 1.27)) hide)
-    )
-  )
   (symbol (lib_id "Device:D_Small") (at 234.696 27.94 270) (unit 1)
     (in_bom yes) (on_board yes)
@@
     )
   )
+  (symbol (lib_id "Device:D_Small") (at 234.696 139.7 270) (unit 1)
+    (in_bom yes) (on_board yes)
+    (property "Reference" "D80" (id 0) (at 236.474 139.7 90)
+      (effects (font (size 0.75 0.75)) (justify left))
+    )
+    (property "Value" "1N4148W" (id 1) (at 236.474 140.849 90)
+      (effects (font (size 0.75 0.75)) (justify left))
+    )
+    (property "Footprint" "acheron_Components:D_SOD-123" (id 2) (at 234.696 139.7 90)
+      (effects (font (size 1.27 1.27)) hide)
+    )
+    (property "Datasheet" "~" (id 3) (at 234.696 139.7 90)
+      (effects (font (size 1.27 1.27)) hide)
+    )
+    (property "MANUFACTURER" "" (id 4) (at 234.696 139.7 90)
+      (effects (font (size 1.27 1.27)) hide)
+    )
+    (property "MANUFACTURER PART NUMBER" "" (id 5) (at 234.696 139.7 90)
+      (effects (font (size 1.27 1.27)) hide)
+    )
+    (property "PACKAGE" "SOD-123" (id 6) (at 234.696 139.7 90)
+      (effects (font (size 1.27 1.27)) hide)
+    )
+    (property "LCSC PART NUMBER" "" (id 7) (at 234.696 139.7 90)
+      (effects (font (size 1.27 1.27)) hide)
+    )
+  )
   (symbol (lib_id "Device:D_Small") (at 255.016 27.94 270) (unit 1)
     (in_bom yes) (on_board yes)
@@
     )
   )
-  (symbol (lib_id "acheronSymbols:MXSwitch") (at 214.376 151.892 0) (unit 1)
-    (in_bom no) (on_board yes)
-    (property "Reference" "SW80" (id 0) (at 214.376 150.622 0))
-    (property "Value" "SPACE" (id 1) (at 214.376 153.162 0)
-      (effects (font (size 0.991 0.991)))
-    )
-    (property "Footprint" "acheron_MX:MX625R" (id 2) (at 214.376 151.892 0)
-      (effects (font (size 1.27 1.27)) hide)
-    )
-    (property "Datasheet" "" (id 3) (at 214.376 151.892 0)
-      (effects (font (size 1.27 1.27)) hide)
-    )
-  )
   (symbol (lib_id "acheronSymbols:MXSwitch") (at 234.696 40.132 0) (unit 1)
     (in_bom no) (on_board yes)
@@
       (effects (font (size 1.27 1.27)) hide)
     )
+  )
+  (symbol (lib_id "acheronSymbols:MXSwitch") (at 234.696 151.892 0) (unit 1)
+    (in_bom no) (on_board yes)
+    (property "Reference" "SW80" (id 0) (at 234.696 150.622 0))
+    (property "Value" "SPACE" (id 1) (at 234.696 153.162 0)
+      (effects (font (size 0.991 0.991)))
+    )
+    (property "Footprint" "acheron_MX:MX625R" (id 2) (at 234.696 151.892 0)
+      (effects (font (size 1.27 1.27)) hide)
+    )
+    (property "Datasheet" "" (id 3) (at 234.696 151.892 0)
+      (effects (font (size 1.27 1.27)) hide)
+    )
