File: Sinister/sinister.kicad_sch (KiCad schematic)
At the start: 426 parts, among them J1 TYPE-C-31-M12_13, J2 Conn_ARM_JTAG_SWD_10, Q1 AO3401A, Q2 DTC123JKAT146, Q3 DTC123JKAT146, Q4 AO3401A, SW1 MINUS, SW10 4, SW11 5, SW12 6, SW13 7, SW14 8, SW15 9, SW16 0, SW17 MINUS, SW18 PLUS, SW19 BKSP, SW2 FSLASH, SW20 NUM 7, SW21 NUM 8, SW22 NUM 9, SW23 END, SW24 TAB, SW25 Q, SW26 W, SW27 E, SW28 R, SW29 T, SW3 ASTERISK, SW30 Y, SW31 U, SW32 I, SW33 O, SW34 P, SW35 LBRKT, SW36 RBRKT, SW37 BSLASH, SW38 NUM PLUS, SW39 NUM4, SW4 NUM LOCK, SW40 NUM5, SW41 NUM 6, SW42 DEL, SW43 CAPSLOCK, SW44 A, SW45 S, SW46 D, SW47 F, SW48 G, SW49 H, SW5 HOME, SW50 J, SW51 K, SW52 L, SW53 COLON, SW54 QUOTE, SW55 ENTER, SW56 NUM 1, SW57 NUM 2, SW58 NUM 3, SW59 UP, SW6 ESC, SW60 LSHIFT, SW61 Z, SW62 X, SW63 C, SW64 V, SW65 B, SW66 N, SW67 M, SW68 COMMA, SW69 PERIOD, SW7 1, SW70 FSLASH, SW71 RSHIFT, SW72 NUM ENTER, SW73 NUM PERIOD, SW74 NUM 0, SW75 LEFT, SW76 DOWN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

Commit message: Rereouted diodes. Placed LED components.
Replaced diodes tracks. Placed and routed LED power components. Routed 5V RGB tracks.
Connections:
- net COL14: no longer SW82.1 (Col)
- net COL15: now also SW82.1 (Col); no longer SW83.1 (Col)
- net COL16: now also SW83.1 (Col); no longer SW84.1 (Col)
- net COL17: now also SW84.1 (Col)
- net LED_PWM: now also U1.16 (PA6/ADC_IN6/TIM3_CH1/TIM16_CH1)
- net Row0 renamed ROW0
Other:
- moved on the sheet: D82, D83, D84, SW82, SW83, SW84
Changed lines of the file:
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@@
   (junction (at 307.086 68.072) (diameter 0) (color 0 0 0 0))
   (junction (at 307.086 96.012) (diameter 0) (color 0 0 0 0))
-  (junction (at 307.086 123.952) (diameter 0) (color 0 0 0 0))
   (junction (at 311.912 227.33) (diameter 0) (color 0 0 0 0))
   (junction (at 315.214 172.974) (diameter 0) (color 0 0 0 0))
@@
   (junction (at 315.976 81.28) (diameter 0) (color 0 0 0 0))
   (junction (at 315.976 109.22) (diameter 0) (color 0 0 0 0))
-  (junction (at 315.976 137.16) (diameter 0) (color 0 0 0 0))
   (junction (at 320.802 227.33) (diameter 0) (color 0 0 0 0))
   (junction (at 324.104 187.706) (diameter 0) (color 0 0 0 0))
@@
   (junction (at 356.616 53.34) (diameter 0) (color 0 0 0 0))
   (junction (at 356.616 81.28) (diameter 0) (color 0 0 0 0))
+  (junction (at 356.616 137.16) (diameter 0) (color 0 0 0 0))
   (junction (at 359.156 227.33) (diameter 0) (color 0 0 0 0))
   (junction (at 368.046 40.132) (diameter 0) (color 0 0 0 0))
   (junction (at 368.046 68.072) (diameter 0) (color 0 0 0 0))
+  (junction (at 368.046 96.012) (diameter 0) (color 0 0 0 0))
   (junction (at 376.936 25.4) (diameter 0) (color 0 0 0 0))
   (junction (at 376.936 53.34) (diameter 0) (color 0 0 0 0))
@@
   (junction (at 528.574 36.576) (diameter 0) (color 0 0 0 0))
   (junction (at 528.574 42.926) (diameter 0) (color 0 0 0 0))
+  (no_connect (at 320.04 278.638))
   (no_connect (at 279.4 233.68))
+  (no_connect (at 320.04 281.178))
   (no_connect (at 517.144 100.076))
   (no_connect (at 227.076 368.046))
-  (no_connect (at 320.04 278.638))
-  (no_connect (at 320.04 281.178))
   (no_connect (at 279.4 231.14))
   (wire (pts (xy 20.32 334.264) (xy 29.21 334.264))
@@
     (stroke (width 0) (type solid) (color 0 0 0 0))
   )
-  (wire (pts (xy 295.656 137.16) (xy 315.976 137.16))
+  (wire (pts (xy 295.656 137.16) (xy 336.296 137.16))
     (stroke (width 0) (type solid) (color 0 0 0 0))
   )
@@
     (stroke (width 0) (type solid) (color 0 0 0 0))
   )
-  (wire (pts (xy 307.086 123.952) (xy 307.086 151.892))
-    (stroke (width 0) (type solid) (color 0 0 0 0))
-  )
   (wire (pts (xy 309.372 227.33) (xy 311.912 227.33))
     (stroke (width 0) (type solid) (color 0 0 0 0))
@@
     (stroke (width 0) (type solid) (color 0 0 0 0))
   )
-  (wire (pts (xy 315.976 137.16) (xy 336.296 137.16))
-    (stroke (width 0) (type solid) (color 0 0 0 0))
-  )
-  (wire (pts (xy 315.976 142.24) (xy 315.976 143.002))
-    (stroke (width 0) (type solid) (color 0 0 0 0))
-  )
   (wire (pts (xy 320.802 227.33) (xy 320.802 229.87))
     (stroke (width 0) (type solid) (color 0 0 0 0))
@@
     (stroke (width 0) (type solid) (color 0 0 0 0))
   )
+  (wire (pts (xy 356.616 137.16) (xy 376.936 137.16))
+    (stroke (width 0) (type solid) (color 0 0 0 0))
+  )
   (wire (pts (xy 356.616 142.24) (xy 356.616 143.002))
     (stroke (width 0) (type solid) (color 0 0 0 0))
@@
     (stroke (width 0) (type solid) (color 0 0 0 0))
   )
+  (wire (pts (xy 368.046 96.012) (xy 368.046 151.892))
+    (stroke (width 0) (type solid) (color 0 0 0 0))
+  )
   (wire (pts (xy 376.936 25.4) (xy 397.256 25.4))
     (stroke (width 0) (type solid) (color 0 0 0 0))
@@
     (stroke (width 0) (type solid) (color 0 0 0 0))
   )
+  (wire (pts (xy 376.936 142.24) (xy 376.936 143.002))
+    (stroke (width 0) (type solid) (color 0 0 0 0))
+  )
   (wire (pts (xy 388.366 24.13) (xy 388.366 40.132))
     (stroke (width 0) (type solid) (color 0 0 0 0))
@@
     (effects (font (size 2.54 2.54)) (justify right bottom))
   )
-  (global_label "Row0" (shape input) (at 21.336 25.4 180)
+  (global_label "ROW0" (shape input) (at 21.336 25.4 180)
     (effects (font (size 0.75 0.75)) (justify right))
   )
@@
     (effects (font (size 1.27 1.27)) (justify left))
   )
+  (global_label "LED_PWM" (shape output) (at 457.454 114.046 270)
+    (effects (font (size 1.27 1.27)) (justify right))
+  )
   (global_label "BOOT0" (shape output) (at 463.804 26.416 90)
     (effects (font (size 1.27 1.27)) (justify left))
@@
     )
   )
-  (symbol (lib_id "Device:D_Small") (at 315.976 139.7 270) (unit 1)
-    (in_bom yes) (on_board yes)
-    (property "Reference" "D82" (id 0) (at 317.754 139.7 90)
-      (effects (font (size 0.75 0.75)) (justify left))
-    )
-    (property "Value" "1N4148W" (id 1) (at 317.754 140.849 90)
-      (effects (font (size 0.75 0.75)) (justify left))
-    )
-    (property "Footprint" "acheron_Components:D_SOD-123" (id 2) (at 315.976 139.7 90)
-      (effects (font (size 1.27 1.27)) hide)
-    )
-    (property "Datasheet" "~" (id 3) (at 315.976 139.7 90)
-      (effects (font (size 1.27 1.27)) hide)
-    )
-    (property "MANUFACTURER" "" (id 4) (at 315.976 139.7 90)
-      (effects (font (size 1.27 1.27)) hide)
-    )
-    (property "MANUFACTURER PART NUMBER" "" (id 5) (at 315.976 139.7 90)
-      (effects (font (size 1.27 1.27)) hide)
-    )
-    (property "PACKAGE" "SOD-123" (id 6) (at 315.976 139.7 90)
-      (effects (font (size 1.27 1.27)) hide)
-    )
-    (property "LCSC PART NUMBER" "" (id 7) (at 315.976 139.7 90)
-      (effects (font (size 1.27 1.27)) hide)
-    )
-  )
   (symbol (lib_id "Device:D_Small") (at 319.024 172.974 180) (unit 1)
     (in_bom yes) (on_board yes)
@@
   (symbol (lib_id "Device:D_Small") (at 336.296 139.7 270) (unit 1)
     (in_bom yes) (on_board yes)
-    (property "Reference" "D83" (id 0) (at 338.074 139.7 90)
+    (property "Reference" "D82" (id 0) (at 338.074 139.7 90)
       (effects (font (size 0.75 0.75)) (justify left))
     )
@@
   (symbol (lib_id "Device:D_Small") (at 356.616 139.7 270) (unit 1)
     (in_bom yes) (on_board yes)
-    (property "Reference" "D84" (id 0) (at 358.394 139.7 90)
+    (property "Reference" "D83" (id 0) (at 358.394 139.7 90)
       (effects (font (size 0.75 0.75)) (justify left))
     )
@@
     )
   )
+  (symbol (lib_id "Device:D_Small") (at 376.936 139.7 270) (unit 1)
+    (in_bom yes) (on_board yes)
+    (property "Reference" "D84" (id 0) (at 378.714 139.7 90)
+      (effects (font (size 0.75 0.75)) (justify left))
+    )
+    (property "Value" "1N4148W" (id 1) (at 378.714 140.849 90)
+      (effects (font (size 0.75 0.75)) (justify left))
+    )
+    (property "Footprint" "acheron_Components:D_SOD-123" (id 2) (at 376.936 139.7 90)
+      (effects (font (size 1.27 1.27)) hide)
+    )
+    (property "Datasheet" "~" (id 3) (at 376.936 139.7 90)
+      (effects (font (size 1.27 1.27)) hide)
+    )
+    (property "MANUFACTURER" "" (id 4) (at 376.936 139.7 90)
+      (effects (font (size 1.27 1.27)) hide)
+    )
+    (property "MANUFACTURER PART NUMBER" "" (id 5) (at 376.936 139.7 90)
+      (effects (font (size 1.27 1.27)) hide)
+    )
+    (property "PACKAGE" "SOD-123" (id 6) (at 376.936 139.7 90)
+      (effects (font (size 1.27 1.27)) hide)
+    )
+    (property "LCSC PART NUMBER" "" (id 7) (at 376.936 139.7 90)
+      (effects (font (size 1.27 1.27)) hide)
+    )
+  )
   (symbol (lib_id "Device:D_Small") (at 397.256 27.94 270) (unit 1)
     (in_bom yes) (on_board yes)
@@
     )
   )
-  (symbol (lib_id "acheronSymbols:MXSwitch") (at 315.976 151.892 0) (unit 1)
-    (in_bom no) (on_board yes)
-    (property "Reference" "SW82" (id 0) (at 315.976 150.622 0))
-    (property "Value" "MENU" (id 1) (at 315.976 153.162 0)
-      (effects (font (size 0.991 0.991)))
-    )
-    (property "Footprint" "acheron_MX:MX125" (id 2) (at 315.976 151.892 0)
-      (effects (font (size 1.27 1.27)) hide)
-    )
-    (property "Datasheet" "" (id 3) (at 315.976 151.892 0)
-      (effects (font (size 1.27 1.27)) hide)
-    )
-  )
   (symbol (lib_id "acheronSymbols:MXSwitch") (at 336.296 40.132 0) (unit 1)
     (in_bom no) (on_board yes)
@@
   (symbol (lib_id "acheronSymbols:MXSwitch") (at 336.296 151.892 0) (unit 1)
     (in_bom no) (on_board yes)
-    (property "Reference" "SW83" (id 0) (at 336.296 150.622 0))
-    (property "Value" "FN" (id 1) (at 336.296 153.162 0)
+    (property "Reference" "SW82" (id 0) (at 336.296 150.622 0))
+    (property "Value" "MENU" (id 1) (at 336.296 153.162 0)
       (effects (font (size 0.991 0.991)))
     )
@@
   (symbol (lib_id "acheronSymbols:MXSwitch") (at 356.616 151.892 0) (unit 1)
     (in_bom no) (on_board yes)
-    (property "Reference" "SW84" (id 0) (at 356.616 150.622 0))
-    (property "Value" "RCRTL" (id 1) (at 356.616 153.162 0)
+    (property "Reference" "SW83" (id 0) (at 356.616 150.622 0))
+    (property "Value" "FN" (id 1) (at 356.616 153.162 0)
       (effects (font (size 0.991 0.991)))
     )
@@
       (effects (font (size 1.27 1.27)) hide)
     )
+  )
+  (symbol (lib_id "acheronSymbols:MXSwitch") (at 376.936 151.892 0) (unit 1)
+    (in_bom no) (on_board yes)
+    (property "Reference" "SW84" (id 0) (at 376.936 150.622 0))
+    (property "Value" "RCRTL" (id 1) (at 376.936 153.162 0)
+      (effects (font (size 0.991 0.991)))
+    )
+    (property "Footprint" "acheron_MX:MX125" (id 2) (at 376.936 151.892 0)
+      (effects (font (size 1.27 1.27)) hide)
+    )
+    (property "Datasheet" "" (id 3) (at 376.936 151.892 0)
+      (effects (font (size 1.27 1.27)) hide)
+    )

Commit message: Began routing Rows and Columns. Added Indicator LEDs.
Finished routing Rows, Halfway through routing Columns. Added and routed Indicator lights for Num Lock, Caps Lock, and Layers 1-3. Added GND and 3V3 pours and islands.
Parts:
- added LED85, LED86, LED87, LED88, LED89: LED, acheron_Components:LED_THT_2.54mm, symbol acheronSymbols:LED
- added R115, R116, R117, R118, R119: 390R, acheron_Components:R_SMD_1206, symbol Device:R_Small
Connections:
- net COL0 is gone; now on net COL1: SW1.1 (Col), SW38.1 (Col), SW72.1 (Col)
- net ROW0 is gone; now on net ROW1: D1.1 (K), D10.1 (K), D11.1 (K), D12.1 (K), D13.1 (K), D14.1 (K), D15.1 (K), D16.1 (K), D17.1 (K), D18.1 (K), D19.1 (K), D2.1 (K), D3.1 (K), D4.1 (K), D5.1 (K), D6.1 (K), D7.1 (K), D8.1 (K), D9.1 (K)
- net COL1: now also U1.17 (PA7/TIM3_CH2/TIM14_CH1/ADC_IN7); no longer SW2.1 (Col), SW20.1 (Col), SW39.1 (Col), SW56.1 (Col), SW73.1 (Col)
- net COL10: now also SW10.1 (Col), SW28.1 (Col), SW47.1 (Col), SW64.1 (Col); no longer SW11.1 (Col), SW29.1 (Col), SW48.1 (Col), SW65.1 (Col), SW80.1 (Col)
- net COL11: now also SW11.1 (Col), SW29.1 (Col), SW48.1 (Col), SW65.1 (Col), SW80.1 (Col); no longer SW12.1 (Col), SW30.1 (Col), SW49.1 (Col), SW66.1 (Col)
- net COL12: now also SW12.1 (Col), SW30.1 (Col), SW49.1 (Col), SW66.1 (Col); no longer SW13.1 (Col), SW31.1 (Col), SW50.1 (Col), SW67.1 (Col)
- net COL13: now also SW13.1 (Col), SW31.1 (Col), SW50.1 (Col), SW67.1 (Col); no longer SW14.1 (Col), SW32.1 (Col), SW51.1 (Col), SW68.1 (Col), SW81.1 (Col)
- net COL14: now also SW14.1 (Col), SW32.1 (Col), SW51.1 (Col), SW68.1 (Col), SW81.1 (Col); no longer SW15.1 (Col), SW33.1 (Col), SW52.1 (Col), SW69.1 (Col)
- net COL15: now also SW15.1 (Col), SW33.1 (Col), SW52.1 (Col), SW69.1 (Col); no longer SW16.1 (Col), SW34.1 (Col), SW53.1 (Col), SW70.1 (Col), SW82.1 (Col)
- net COL16: now also SW16.1 (Col), SW34.1 (Col), SW53.1 (Col), SW70.1 (Col), SW82.1 (Col); no longer SW17.1 (Col), SW35.1 (Col), SW54.1 (Col), SW71.1 (Col), SW83.1 (Col)
- net COL17: now also SW17.1 (Col), SW35.1 (Col), SW54.1 (Col), SW71.1 (Col), SW83.1 (Col); no longer SW18.1 (Col), SW36.1 (Col), SW55.1 (Col), SW84.1 (Col)
- net COL18: now also SW18.1 (Col), SW36.1 (Col), SW55.1 (Col), SW84.1 (Col); no longer SW19.1 (Col), SW37.1 (Col)
- net COL2: now also SW2.1 (Col), SW20.1 (Col), SW39.1 (Col), SW56.1 (Col), SW73.1 (Col), U1.18 (PB0/TIM3_CH3/ADC_IN8); no longer SW21.1 (Col), SW3.1 (Col), SW40.1 (Col), SW57.1 (Col), SW74.1 (Col)
- net COL3: now also SW21.1 (Col), SW3.1 (Col), SW40.1 (Col), SW57.1 (Col), SW74.1 (Col), U1.19 (PB1/TIM3_CH4/TIM14_CH1/ADC_IN9); no longer SW22.1 (Col), SW4.1 (Col), SW41.1 (Col), SW58.1 (Col), SW75.1 (Col)
- net COL4: now also SW22.1 (Col), SW4.1 (Col), SW41.1 (Col), SW58.1 (Col), SW75.1 (Col), U1.20 (PB2); no longer SW23.1 (Col), SW42.1 (Col), SW5.1 (Col), SW59.1 (Col), SW76.1 (Col)
- net COL5: now also SW23.1 (Col), SW42.1 (Col), SW5.1 (Col), SW59.1 (Col), SW76.1 (Col), U1.21 (PB10/SPI2_SCK/I2C2_SCL/TIM2_CH3); no longer SW24.1 (Col), SW43.1 (Col), SW6.1 (Col), SW60.1 (Col), SW77.1 (Col)
- net COL6: now also SW24.1 (Col), SW43.1 (Col), SW6.1 (Col), SW60.1 (Col), SW77.1 (Col), U1.31 (TIM1_CH3/PA10); no longer SW25.1 (Col), SW44.1 (Col), SW61.1 (Col), SW7.1 (Col), SW78.1 (Col)
- net COL7: now also SW25.1 (Col), SW44.1 (Col), SW61.1 (Col), SW7.1 (Col), SW78.1 (Col), U1.10 (PA0/ADC_IN0); no longer SW26.1 (Col), SW45.1 (Col), SW62.1 (Col), SW79.1 (Col), SW8.1 (Col)
- net COL8: now also SW26.1 (Col), SW45.1 (Col), SW62.1 (Col), SW79.1 (Col), SW8.1 (Col), U1.11 (PA1/ADC_IN1); no longer SW27.1 (Col), SW46.1 (Col), SW63.1 (Col), SW9.1 (Col)
- net COL9: now also SW27.1 (Col), SW46.1 (Col), SW63.1 (Col), SW9.1 (Col), U1.12 (PA2/ADC_IN2); no longer SW10.1 (Col), SW28.1 (Col), SW47.1 (Col), SW64.1 (Col)
- net GND: now also LED85.K, LED86.K, LED87.K, LED88.K, LED89.K
- net ROW1: now also U1.29 (TIM1_CH1/PA8); no longer D20.1 (K), D21.1 (K), D22.1 (K), D23.1 (K), D24.1 (K), D25.1 (K), D26.1 (K), D27.1 (K), D28.1 (K), D29.1 (K), D30.1 (K), D31.1 (K), D32.1 (K), D33.1 (K), D34.1 (K), D35.1 (K), D36.1 (K), D37.1 (K)
- net ROW2: now also D20.1 (K), D21.1 (K), D22.1 (K), D23.1 (K), D24.1 (K), D25.1 (K), D26.1 (K), D27.1 (K), D28.1 (K), D29.1 (K), D30.1 (K), D31.1 (K), D32.1 (K), D33.1 (K), D34.1 (K), D35.1 (K), D36.1 (K), D37.1 (K), U1.30 (TIM1_CH2/PA9); no longer D38.1 (K), D39.1 (K), D40.1 (K), D41.1 (K), D42.1 (K), D43.1 (K), D44.1 (K), D45.1 (K), D46.1 (K), D47.1 (K), D48.1 (K), D49.1 (K), D50.1 (K), D51.1 (K), D52.1 (K), D53.1 (K), D54.1 (K), D55.1 (K)
- net ROW3: now also D38.1 (K), D39.1 (K), D40.1 (K), D41.1 (K), D42.1 (K), D43.1 (K), D44.1 (K), D45.1 (K), D46.1 (K), D47.1 (K), D48.1 (K), D49.1 (K), D50.1 (K), D51.1 (K), D52.1 (K), D53.1 (K), D54.1 (K), D55.1 (K), U1.22 (PB11/TIM2_CH4/I2C2_SDA); no longer D56.1 (K), D57.1 (K), D58.1 (K), D59.1 (K), D60.1 (K), D61.1 (K), D62.1 (K), D63.1 (K), D64.1 (K), D65.1 (K), D66.1 (K), D67.1 (K), D68.1 (K), D69.1 (K), D70.1 (K), D71.1 (K)
- net ROW4: now also D56.1 (K), D57.1 (K), D58.1 (K), D59.1 (K), D60.1 (K), D61.1 (K), D62.1 (K), D63.1 (K), D64.1 (K), D65.1 (K), D66.1 (K), D67.1 (K), D68.1 (K), D69.1 (K), D70.1 (K), D71.1 (K), U1.5 (PF0/OSC_IN); no longer D72.1 (K), D73.1 (K), D74.1 (K), D75.1 (K), D76.1 (K), D77.1 (K), D78.1 (K), D79.1 (K), D80.1 (K), D81.1 (K), D82.1 (K), D83.1 (K), D84.1 (K)
- net INDICATOR3: now reaches U1.13 (PA3/TIM15_CH2/ADC_IN3)
- net INDICATOR3: now also R117.2
- net INDICATOR4: now reaches U1.14 (PA4/TIM14_CH1/ADC_IN4)
- net INDICATOR4: now also R118.2
- net INDICATOR5: now reaches U1.15 (PA5/ADC_IN5/DAC_OUT2)
- net INDICATOR5: now also R119.2
- net INDICATOR1: now reaches U1.25 (PB12)
- net INDICATOR1: now also R115.2
- net INDICATOR2: now reaches U1.27 (SPI2_MISO/I2S2_MCK/I2C2_SDA/TIM15_CH1/PB14)
- net INDICATOR2: now also R116.2
- net ROW5: now reaches U1.6 (PF1/OSC_OUT)
- net ROW5: now also D72.1 (K), D73.1 (K), D74.1 (K), D75.1 (K), D76.1 (K), D77.1 (K), D78.1 (K), D79.1 (K), D80.1 (K), D81.1 (K), D82.1 (K), D83.1 (K), D84.1 (K)
- new net: LED86.A, R116.1
- new net: LED87.A, R117.1
- new net: LED89.A, R119.1
- new net: LED88.A, R118.1
- new net: LED85.A, R115.1
- new net COL19: SW19.1 (Col), SW37.1 (Col)
Other:
- note added: "INDICATOR LEDs"
