File: Sinister/sinister.kicad_sch (KiCad schematic)
At the start: 436 parts, among them J1 TYPE-C-31-M12_13, J2 Conn_ARM_JTAG_SWD_10, Q1 AO3401A, Q2 DTC123JKAT146, Q3 DTC123JKAT146, Q4 AO3401A, SW1 MINUS, SW10 4, SW11 5, SW12 6, SW13 7, SW14 8, SW15 9, SW16 0, SW17 MINUS, SW18 PLUS, SW19 BKSP, SW2 FSLASH, SW20 NUM 7, SW21 NUM 8, SW22 NUM 9, SW23 END, SW24 TAB, SW25 Q, SW26 W, SW27 E, SW28 R, SW29 T, SW3 ASTERISK, SW30 Y, SW31 U, SW32 I, SW33 O, SW34 P, SW35 LBRKT, SW36 RBRKT, SW37 BSLASH, SW38 NUM PLUS, SW39 NUM4, SW4 NUM LOCK, SW40 NUM5, SW41 NUM 6, SW42 DEL, SW43 CAPSLOCK, SW44 A, SW45 S, SW46 D, SW47 F, SW48 G, SW49 H, SW5 HOME, SW50 J, SW51 K, SW52 L, SW53 COLON, SW54 QUOTE, SW55 ENTER, SW56 NUM 1, SW57 NUM 2, SW58 NUM 3, SW59 UP, SW6 ESC, SW60 LSHIFT, SW61 Z, SW62 X, SW63 C, SW64 V, SW65 B, SW66 N, SW67 M, SW68 COMMA, SW69 PERIOD, SW7 1, SW70 FSLASH, SW71 RSHIFT, SW72 NUM ENTER, SW73 NUM PERIOD, SW74 NUM 0, SW75 LEFT, SW76 DOWN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

Commit message: Repaired Logo. Added Solenoid.
Repaired problematic polygons on the Logo that were causing incorrect line thickness during loads from save file. Added and routed components for external solenoid. Finished BOM xlsx.
Parts:
- added D104: 1N4001W, Diode_SMD:D_SOD-123F, symbol Device:D_Small
- added J3: DC-003-2A-1.3, acheron_Connectors:CUI_PJ-036C, symbol Connector:Barrel_Jack_Switch
- added Q5: MJD122T4G, acheron_Components:DPAK229P990X238-3N, symbol Device:Q_NPN_Darlington_BCE
- added R120: 1k, acheron_Components:R_SMD_1206, symbol Device:R_Small
- D100, D101, D102, D103, D88, D89, D90, D91, D92, D93, D94, D95, D96, D97, D98, D99: LCSC PART NUMBER (none) -> C114587; LCSC PART NUMBER\ C114587 -> (none)
- F1: MANUFACTURER Littelfuse -> (none)
- LED1, LED10, LED11, LED12, LED13, LED14, LED15, LED16, LED17, LED18, LED19, LED2, LED20, LED21, LED22, LED23, LED24, LED25, LED26, LED27, LED28, LED29, LED3, LED30, LED31, LED32, LED33, LED34, LED35, LED36, LED37, LED38, LED39, LED4, LED40, LED41, LED42, LED43, LED44, LED45, LED46, LED47, LED48, LED49, LED5, LED50, LED51, LED52, LED53, LED54, LED55, LED56, LED57, LED58, LED59, LED6, LED60, LED61, LED62, LED63, LED64, LED65, LED66, LED67, LED68, LED69, LED7, LED70, LED71, LED72, LED73, LED74, LED75, LED76, LED77, LED78, LED79, LED8, LED80, LED81, LED82, LED83, LED84, LED9: now left out of the parts list
Connections:
- net 5V: now also D104.1 (K), J3.2
- net GND: now also Q5.3 (E)
- net SHIELD: now reaches C13.1, C14.1, J1.S (SHIELD), R65.2, R66.2
- net SOLENOID: now reaches U1.38 (PA15)
- net SOLENOID: now also R120.2
- new net: D104.2 (A), J3.1, J3.3, Q5.2 (C)
- new net: Q5.1 (B), R120.1
- no-connect marks 7 -> 6
Other:
- note added: "SOLENOID"
